File: Tiny_Solar_Supply.kicad_pcb (KiCad board)
At the start: 2 copper layers, 42.5 x 20.3 mm, 18 parts, among them J1 Conn_01x02, J2 Conn_01x02, J3 Conn_01x02, J4 Conn_01x02, Q1 2N7002, U1 AP3015AKTR-G1

Commit message: Gerber files generated
Routing:
- net /OUT_P: track 32.9 -> 32.3 mm
Changed lines of the file:
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@@
 			(plot_on_all_layers_selection 0x00000000_00000000_00000000_00000000)
 			(disableapertmacros no)
-			(usegerberextensions no)
+			(usegerberextensions yes)
 			(usegerberattributes yes)
 			(usegerberadvancedattributes yes)
@@
 			(outputformat 1)
 			(mirror no)
-			(drillshape 1)
+			(drillshape 0)
 			(scaleselection 1)
-			(outputdirectory "")
+			(outputdirectory "Gerber/")
 		)
 	)
@@
 	)
 	(segment
-		(start 164.2364 55.9308)
-		(end 161.854261 55.9308)
+		(start 164.465 53.523731)
+		(end 164.465 55.245)
 		(width 0.25)
 		(layer "F.Cu")
@@
 	)
 	(segment
-		(start 165.419376 52.569355)
-		(end 164.2364 53.752331)
+		(start 175.959954 50.23742)
+		(end 175.959954 54.265646)
 		(width 0.25)
 		(layer "F.Cu")
@@
 	)
 	(segment
-		(start 175.959954 50.23742)
-		(end 175.959954 54.265646)
+		(start 168.3512 55.5244)
+		(end 169.376857 56.550057)
 		(width 0.25)
 		(layer "F.Cu")
@@
 	)
 	(segment
-		(start 168.3512 55.5244)
-		(end 169.376857 56.550057)
+		(start 165.419376 52.569355)
+		(end 166.615355 52.569355)
 		(width 0.25)
 		(layer "F.Cu")
@@
 	)
 	(segment
-		(start 165.419376 52.569355)
-		(end 166.615355 52.569355)
+		(start 175.959954 54.265646)
+		(end 173.675543 56.550057)
 		(width 0.25)
 		(layer "F.Cu")
@@
 	)
 	(segment
-		(start 175.959954 54.265646)
-		(end 173.675543 56.550057)
+		(start 163.7792 55.9308)
+		(end 161.854261 55.9308)
 		(width 0.25)
 		(layer "F.Cu")
@@
 	)
 	(segment
-		(start 164.2364 53.752331)
-		(end 164.2364 55.9308)
+		(start 165.419376 52.569355)
+		(end 164.465 53.523731)
+		(width 0.25)
+		(layer "F.Cu")
+		(net 2)
+	)
+	(segment
+		(start 164.465 55.245)
+		(end 163.7792 55.9308)
 		(width 0.25)
 		(layer "F.Cu")
@@
 	)
 	(segment
-		(start 177.5968 56.825466)
-		(end 179.635516 54.78675)
+		(start 177.5968 59.8932)
+		(end 177.5968 56.825466)
 		(width 0.35)
 		(layer "F.Cu")
@@
 	)
 	(segment
+		(start 173.540179 62.792159)
+		(end 173.540179 61.206621)
+		(width 0.35)
+		(layer "F.Cu")
+		(net 3)
+	)
+	(segment
+		(start 173.8884 60.8584)
+		(end 176.6316 60.8584)
+		(width 0.35)
+		(layer "F.Cu")
+		(net 3)
+	)
+	(segment
 		(start 168.818987 57.922587)
 		(end 168.818987 58.666023)
@@
 	)
 	(segment
-		(start 173.8884 60.8584)
-		(end 177.5968 60.8584)
+		(start 177.5968 56.825466)
+		(end 179.635516 54.78675)
 		(width 0.35)
 		(layer "F.Cu")
@@
 	)
 	(segment
-		(start 177.5968 60.8584)
-		(end 177.5968 56.825466)
+		(start 176.6316 60.8584)
+		(end 177.5968 59.8932)
 		(width 0.35)
 		(layer "F.Cu")
@@
 		(width 0.35)
 		(layer "F.Cu")
-		(net 3)
-	)
-	(segment
-		(start 173.540179 62.792159)
-		(end 173.540179 61.206621)
-		(width 0.35)
-		(layer "F.Cu")
